File: hackpad/hackpad.kicad_pcb (KiCad board)
At the start: 2 copper layers, 95.3 x 88.4 mm, 21 parts, among them SW1 SW_Push_45deg, SW10 RotaryEncoder_Switch, SW2 SW_Push_45deg, SW3 SW_Push_45deg, SW4 SW_Push_45deg, SW5 SW_Push_45deg, SW6 SW_Push_45deg, SW7 SW_Push_45deg, SW8 SW_Push_45deg, SW9 SW_Push_45deg, U1 MOUDLE-SEEEDUINO-XIAO, U2 ER_OLEDM0.91_1x-I2C

Commit message: rotated XIAO
Parts:
- SW10: value RotaryEncoder_Switch -> RotaryEncoder_Switch_MP
- moved U1 2.34 mm to (111.4, 71.3), turned to -90 degrees
- moved SW10 0.06 mm to (39.4, 34.5)
Connections:
- SW10 pad MP: (no net) -> GND
Routing:
- net GND: track 140.9 -> 277.5 mm
- net Net-(U1-PA5_A9_D9_MISO): track 114.5 -> 214.2 mm, vias 0 -> 4
- net Net-(U1-PB08_A6_D6_TX): track 164.7 -> 114.5 mm
- net Row 2: track 58.7 -> 92.7 mm, vias 0 -> 2
- net Column 0: track 99.1 -> 128.8 mm
- net Net-(U1-PB09_A7_D7_RX): track 180.9 -> 159.9 mm
- net Column 1: track 86.4 -> 105.5 mm, vias 4 -> 0
- net Net-(U1-PA6_A10_D10_MOSI): track 103.3 -> 116.9 mm, vias 2 -> 4
- net Row 1: track 57.1 -> 68.3 mm, vias 0 -> 1
- net Net-(U1-3V3): track 116.9 -> 109.4 mm
- net Column 2: track 75.1 -> 82.6 mm, vias 2 -> 0
- net Net-(U1-PA7_A8_D8_SCK): track 115.0 -> 120.8 mm
- net Row 0: track 70.6 -> 69.6 mm, vias 0 -> 2
