File: PCB/smolpad.kicad_pcb (KiCad board)
At the start: 2 copper layers, 95.3 x 88.4 mm, 26 parts, among them SW1 SW_Push_45deg, SW10 RotaryEncoder_Switch_MP, SW2 SW_Push_45deg, SW3 SW_Push_45deg, SW4 SW_Push_45deg, SW5 SW_Push_45deg, SW6 SW_Push_45deg, SW7 SW_Push_45deg, SW8 SW_Push_45deg, SW9 SW_Push_45deg, U1 MOUDLE-SEEEDUINO-XIAO, U2 ER_OLEDM0.91_1x-I2C

Commit message: changed footprints
Parts:
- SW1, SW2, SW3, SW4, SW5, SW6, SW7, SW8, SW9: value SW_Push_45deg -> SW_Push; footprint Button_Switch_Keyboard:SW_Cherry_MX_1.00u_Plate -> Button_Switch_Keyboard:SW_Cherry_MX_1.00u_PCB
- moved SW8 0.22 mm to (69.2, 88.0)
Routing:
- net Net-(D2-A): track 15.4 -> 17.8 mm
- net Net-(D3-A): track 15.4 -> 17.9 mm
